File: Pruebas/Prueba_placa_potencia/Prueba_placa_potencia.kicad_sch (KiCad schematic)
At the start: 51 parts, among them J1 Screw_Terminal_01x02, J2 Screw_Terminal_01x02, J3 Screw_Terminal_01x02, J4 Conn_01x03_Pin, J5 Conn_01x03_Pin, J6 Conn_01x03_Pin, J7 Conn_01x01_Pin, J8 Conn_01x01_Pin, Q1 TIP142, Q10 TIP142, Q11 2N2222A, Q2 2N2222A, Q3 2N2222A, Q4 TIP142, Q5 2N2222A, Q6 TIP142, Q7 2N2222A, Q8 TIP142, Q9 2N2222A, U1 LM358

Commit message: Esquemático listo
Parts:
- removed D2: BZX85C3V3, BZX85C3V3:DIOAD1036W73L450D282, symbol BZX85C3V3:BZX85C3V3
- removed J2, J3: Screw_Terminal_01x02, symbol Connector:Screw_Terminal_01x02
- removed Q1, Q10, Q4, Q6, Q8: TIP142, TIP142:SOT93, symbol TIP142:TIP142
- removed VR1: 3296W-1-103ALF, 3296W-1-103ALF:TRIM_3296W-1-103ALF, symbol 3296W-1-103ALF:3296W-1-103ALF
- added C2: 100u, Capacitor_THT:CP_Radial_D5.0mm_P2.00mm, symbol Device:C_Polarized
- added C3: 10u, Capacitor_THT:CP_Radial_D5.0mm_P2.00mm, symbol Device:C_Polarized
- added C4: 100n, Capacitor_THT:C_Disc_D5.0mm_W2.5mm_P2.50mm, symbol Device:C
- added D3: BZX85C3V3, Diode_THT:D_T-1_P5.08mm_Horizontal, symbol Device:D_Zener
- added J4: Screw_Terminal_01x02, TerminalBlock_4Ucon:TerminalBlock_4Ucon_1x02_P3.50mm_Horizontal, symbol Connector:Screw_Terminal_01x02
- added Q11, Q3, Q5, Q7, Q9: TIP142, Package_TO_SOT_THT:TO-247-3_Horizontal_TabUp, symbol Transistor_BJT:Q_NPN_Darlington_BCE
- added R28: 360, Resistor_THT:R_Axial_DIN0207_L6.3mm_D2.5mm_P7.62mm_Horizontal, symbol Device:R
- added RV1: 10k, Potentiometer_THT:Potentiometer_Alps_RK09Y11_Single_Horizontal, symbol Device:R_Potentiometer
- C1: footprint (none) -> Capacitor_THT:C_Disc_D5.0mm_W2.5mm_P2.50mm
- D2: renamed from D1; footprint (none) -> LED_THT:LED_D3.0mm
- J3: renamed from J1; footprint (none) -> TerminalBlock_4Ucon:TerminalBlock_4Ucon_1x02_P3.50mm_Horizontal
- J7: value Conn_01x01_Pin -> LOAD+; footprint (none) -> MountingHole:MountingHole_4.3mm_M4_DIN965_Pad
- J8: value Conn_01x01_Pin -> LOAD-; footprint (none) -> MountingHole:MountingHole_4.3mm_M4_DIN965_Pad
- Q1: renamed from Q11; footprint 2N2222A:TO92254P470H750-3 -> Package_TO_SOT_THT:TO-92_Inline
- Q10: renamed from Q9; footprint 2N2222A:TO92254P470H750-3 -> Package_TO_SOT_THT:TO-92_Inline
- Q2: renamed from Q7; footprint 2N2222A:TO92254P470H750-3 -> Package_TO_SOT_THT:TO-92_Inline
- Q4: renamed from Q5; footprint 2N2222A:TO92254P470H750-3 -> Package_TO_SOT_THT:TO-92_Inline
- Q6: renamed from Q2; footprint 2N2222A:TO92254P470H750-3 -> Package_TO_SOT_THT:TO-92_Inline
- Q8: renamed from Q3; footprint 2N2222A:TO92254P470H750-3 -> Package_TO_SOT_THT:TO-92_Inline
- R11: renamed from R33; footprint (none) -> Resistor_THT:R_Axial_DIN0207_L6.3mm_D2.5mm_P7.62mm_Horizontal
- R12: renamed from R24; footprint (none) -> Resistor_THT:R_Axial_DIN0207_L6.3mm_D2.5mm_P7.62mm_Horizontal
- R14: renamed from R17; footprint (none) -> Resistor_THT:R_Axial_DIN0207_L6.3mm_D2.5mm_P7.62mm_Horizontal
- U1: footprint (none) -> Package_DIP:DIP-8_W7.62mm_Socket
- renumbered J5 to J1, J6 to J2, J4 to J6, R21 to R1, R11 to R13, R2 to R15, R1 to R16, R3 to R17, R5 to R18, R4 to R19, R20 to R2, R6 to R20, R8 to R21, R7 to R22, R9 to R23, R12 to R24, R13 to R25, R14 to R26, R15 to R27, R22 to R3, R19 to R4, R26 to R5, R25 to R6, R27 to R7, R18 to R8, R16 to R9
Connections:
- net GND: now also U1.4 (V-), C2.2, C3.2, C4.2, D3.2 (A), R28.2; no longer J8.1 (Pin_1)
- net at Q4.2, R17.1, R18.1: now also Q11.3 (E)
- net E: now reaches J7.1 (Pin_1), R13.2, R15.2, R17.2, R18.2, R20.2, R21.2, R23.2, R24.2, R26.2, R27.2
- net E: now also R8.2; no longer Q1.3, Q10.1, Q2.1, Q4.1, Q6.1, Q8.1
- net B: now reaches R10.1, R16.1, R19.1, R22.1, R25.1
- net B: now also C1.1, U1.1; no longer R1.1, R2.1, R3.1, R8.2, R9.1
- net at Q2.3, R10.2: now also Q3.1 (B)
- net at Q10.3, R25.2: now also Q5.1 (B)
- net at Q10.2, R26.1, R27.1: now also Q5.3 (E)
- net at Q8.2, R23.1, R24.1: now also Q7.3 (E)
- net at Q6.2, R20.1, R21.1: now also Q9.3 (E)
- net at Q8.3, R22.2: now also Q7.1 (B)
- net at R1.2, R2.2, R3.2: now also J1.2 (Pin_2), D3.1 (K); no longer J1.3 (Pin_3)
- net at J2.2 (Pin_2): now also U1.3 (+), RV1.1, RV1.2; no longer R6.2
- net at J2.3 (Pin_3): now also R6.2; no longer U1.3 (+)
- net at Q6.3, R19.2: now also Q9.1 (B)
- net at R6.1: now also J1.3 (Pin_3); no longer J1.2 (Pin_2)
- net VCC: now reaches J3.1 (Pin_1), U1.8 (V+)
- net VCC: now also R1.1, R2.1, R3.1, R9.1, C2.1, C3.1, C4.1
- net at Q4.3, R16.2: now also Q11.1 (B)
- net at Q2.2, R13.1, R15.1: now also Q3.3 (E)
- new net: Q1.3, Q10.1, Q2.1, Q4.1, Q6.1
- new net: R28.1, RV1.3
- new net SRC+: J4.1 (Pin_1), Q11.2 (C), Q3.2 (C), Q5.2 (C), Q7.2 (C), Q9.2 (C)
- new net SRC-: J4.2 (Pin_2), J8.1 (Pin_1)
Other:
- moved on the sheet: C1, J3, J7, R6, U1C
