File: PowerPCB/PowerPCB.kicad_sch (KiCad schematic)
At the start: 81 parts, among them J1 Battery, J10 Conn_01x02, J2 Conn_01x02, J3 12Vout, J4 Conn_01x03, J5 5Vout, J6 Conn_01x03, J7 Conn_01x03, J8 Conn_01x02, J9 Conn_01x03, U1 TPS551892QWRYQRQ1, U2 FS1403-5000-AL

Commit message: minor fixes
Parts:
- J1, J3: footprint TerminalBlock_4Ucon:TerminalBlock_4Ucon_1x02_P3.50mm_Horizontal -> TerminalBlock_MetzConnect:TerminalBlock_MetzConnect_Type094_RT03502HBLU_1x02_P5.00mm_Horizontal
- J5: footprint Connector_PinHeader_2.54mm:PinHeader_1x02_P2.54mm_Vertical -> TerminalBlock_MetzConnect:TerminalBlock_MetzConnect_Type094_RT03502HBLU_1x02_P5.00mm_Horizontal
Changed lines of the file:
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@@
 			)
 		)
-		(property "Footprint" "TerminalBlock_4Ucon:TerminalBlock_4Ucon_1x02_P3.50mm_Horizontal"
+		(property "Footprint" "TerminalBlock_MetzConnect:TerminalBlock_MetzConnect_Type094_RT03502HBLU_1x02_P5.00mm_Horizontal"
 			(at 196.85 92.71 0)
 			(effects
@@
 			)
 		)
-		(property "Footprint" "Connector_PinHeader_2.54mm:PinHeader_1x02_P2.54mm_Vertical"
+		(property "Footprint" "TerminalBlock_MetzConnect:TerminalBlock_MetzConnect_Type094_RT03502HBLU_1x02_P5.00mm_Horizontal"
 			(at 196.85 110.49 0)
 			(effects
@@
 			)
 		)
-		(property "Footprint" "TerminalBlock_4Ucon:TerminalBlock_4Ucon_1x02_P3.50mm_Horizontal"
+		(property "Footprint" "TerminalBlock_MetzConnect:TerminalBlock_MetzConnect_Type094_RT03502HBLU_1x02_P5.00mm_Horizontal"
 			(at 196.85 100.33 0)
 			(effects

Commit message: PowerPCB v2
Parts:
- removed J6: Conn_01x03, Connector_PinHeader_2.54mm:PinHeader_1x03_P2.54mm_Vertical, symbol Connector_Generic:Conn_01x03
- removed R10: 10, Resistor_SMD:R_0805_2012Metric_Pad1.20x1.40mm_HandSolder, symbol Device:R_US
- removed R14: 47k, Resistor_SMD:R_0805_2012Metric_Pad1.20x1.40mm_HandSolder, symbol Device:R_US
- removed R19, R20, R23: 100k, Resistor_SMD:R_0805_2012Metric_Pad1.20x1.40mm_HandSolder, symbol Device:R_US
- removed R24: 0, Resistor_SMD:R_0805_2012Metric_Pad1.20x1.40mm_HandSolder, symbol POWER_STRIP_DESIGN_WITH_ORIGINAL-lib:R
- removed R6: 5.6k, Resistor_SMD:R_1206_3216Metric_Pad1.30x1.75mm_HandSolder, symbol Device:R_US
- removed R7: 2.2k, Resistor_SMD:R_0805_2012Metric_Pad1.20x1.40mm_HandSolder, symbol Device:R_US
- removed TP4, TP5, TP9: TestPoint, TestPoint:TestPoint_Keystone_5019_Miniature, symbol Connector:TestPoint
- added C33: 68uF, Capacitor_SMD:CP_Elec_8x10, symbol Device:C_Polarized_US
- added C34: 0.1uF, Capacitor_SMD:C_0402_1005Metric, symbol Device:C
- added C35: 1uF, Capacitor_SMD:C_0603_1608Metric, symbol Device:C
- added R16: 0, Resistor_SMD:R_0402_1005Metric, symbol Device:R_US
- added R8: 10, Resistor_SMD:R_0402_1005Metric, symbol Device:R_US
- added TP3: TestPoint, TestPoint:TestPoint_Keystone_5019_Miniature, symbol Connector:TestPoint
- C1, C23, C25, C31: footprint Capacitor_SMD:C_0805_2012Metric_Pad1.18x1.45mm_HandSolder -> Capacitor_SMD:C_0402_1005Metric; LCSC (none) -> C248318; Manufacturer (none) -> TDK; PartNumber (none) -> CGA2B3X7R1H103K050BB
- C10, C11, C12, C18, C19: footprint Capacitor_SMD:C_0805_2012Metric_Pad1.18x1.45mm_HandSolder -> Capacitor_SMD:C_1206_3216Metric; LCSC (none) -> C342827; Manufacturer (none) -> TDK; PartNumber (none) -> CGA5L1X7R1H106K160AC
- C13, C16, C20: footprint Capacitor_SMD:C_1206_3216Metric_Pad1.33x1.80mm_HandSolder -> Capacitor_SMD:C_0603_1608Metric; LCSC (none) -> C3011671; Manufacturer (none) -> MuRata; PartNumber (none) -> GRT188R61H105ME13D
- C14, C15, C21, C22: footprint Capacitor_SMD:C_1206_3216Metric_Pad1.33x1.80mm_HandSolder -> Capacitor_SMD:C_0402_1005Metric; LCSC (none) -> C77020; Manufacturer (none) -> MuRata; PartNumber (none) -> GRM155R71H104KE14D
- C17: LCSC (none) -> C542443; Manufacturer (none) -> Panasonic; PartNumber (none) -> EEHZA1H680P
- C2, C24, C28, C6: footprint Capacitor_SMD:C_1206_3216Metric_Pad1.33x1.80mm_HandSolder -> Capacitor_SMD:C_0402_1005Metric; LCSC (none) -> C361198; Manufacturer (none) -> TDK; PartNumber (none) -> C1005X7R1H104KT000F
- C26, C27, C29, C30: footprint Capacitor_SMD:C_0805_2012Metric_Pad1.18x1.45mm_HandSolder -> Capacitor_SMD:C_1206_3216Metric; LCSC (none) -> C2182087; Manufacturer (none) -> TDK; PartNumber (none) -> CGA5L1X7S1A226M160AC
- C3, C4: footprint Capacitor_SMD:C_1206_3216Metric_Pad1.33x1.80mm_HandSolder -> Capacitor_SMD:C_0603_1608Metric; LCSC (none) -> C161181; Manufacturer (none) -> Murata Electronics North America; PartNumber (none) -> GCM188L81H104KA57D
- C32: footprint Capacitor_SMD:C_0805_2012Metric_Pad1.18x1.45mm_HandSolder -> Capacitor_SMD:C_1206_3216Metric; LCSC (none) -> C5449010; Manufacturer (none) -> CCTC; PartNumber (none) -> TCC1206X7R225M250HT
- C5: footprint Capacitor_SMD:C_1206_3216Metric_Pad1.33x1.80mm_HandSolder -> Capacitor_SMD:C_0603_1608Metric; LCSC (none) -> C437574; Manufacturer (none) -> MuRata; PartNumber (none) -> GRT188R61C475KE13D
- C7: footprint Capacitor_SMD:C_0805_2012Metric_Pad1.18x1.45mm_HandSolder -> Capacitor_SMD:C_0402_1005Metric; LCSC (none) -> C2162824; Manufacturer (none) -> TDK; PartNumber (none) -> CGA2B2C0G1H101J050BA
- C8: footprint Capacitor_SMD:C_1206_3216Metric_Pad1.33x1.80mm_HandSolder -> Capacitor_SMD:C_0402_1005Metric; LCSC (none) -> C694277; Manufacturer (none) -> TDK; PartNumber (none) -> C1005X7R1H472KT000F
- C9: footprint Capacitor_SMD:CP_Elec_6.3x5.4 -> Capacitor_SMD:CP_Elec_6.3x5.8; LCSC (none) -> C454360; Manufacturer (none) -> Panasonic; PartNumber (none) -> EEHZK1V101XP
- J1, J5: LCSC (none) -> C7498454; Manufacturer (none) -> DORABO; PartNumber (none) -> DB102-5.0-2P-BU-S
- J10, J2, J8: LCSC (none) -> C52016390; Manufacturer (none) -> hanxia; PartNumber (none) -> HX PH254-01-02-Z-L11.5 male header connector
- J3: renamed from J4; LCSC (none) -> C52016391; Manufacturer (none) -> hanxia; PartNumber (none) -> HX PH254-01-03-Z-L11.5 pcb pin header
- J4: renamed from J3; LCSC (none) -> C7498454; Manufacturer (none) -> DORABO; PartNumber (none) -> DB102-5.0-2P-BU-S
- J7, J9: LCSC (none) -> C52016391; Manufacturer (none) -> hanxia; PartNumber (none) -> HX PH254-01-03-Z-L11.5 pcb pin header
- L1: LCSC (none) -> C3911513; Manufacturer (none) -> Coilcraft; PartNumber (none) -> XAL7070-472MEB
- R1: value 51 -> 49.9; footprint Resistor_SMD:R_0805_2012Metric_Pad1.20x1.40mm_HandSolder -> Resistor_SMD:R_0402_1005Metric; LCSC (none) -> C482189; Manufacturer (none) -> Vishay-Dale; PartNumber (none) -> CRCW040249R9FKED
- R10: renamed from R13; value 100k -> 147k; footprint Resistor_SMD:R_0805_2012Metric_Pad1.20x1.40mm_HandSolder -> Resistor_SMD:R_0402_1005Metric; LCSC (none) -> C2933073; Manufacturer (none) -> FOJAN; PartNumber (none) -> FRC0402F1473TS
- R11: renamed from R16; value 100k -> 115k; footprint Resistor_SMD:R_0805_2012Metric_Pad1.20x1.40mm_HandSolder -> Resistor_SMD:R_0402_1005Metric; LCSC (none) -> C2076632; Manufacturer (none) -> Vishay-Dale; PartNumber (none) -> CRCW0402115KFKED
- R12, R2: value 100k -> 102k; footprint Resistor_SMD:R_0805_2012Metric_Pad1.20x1.40mm_HandSolder -> Resistor_SMD:R_0402_1005Metric; LCSC (none) -> C481920; Manufacturer (none) -> Vishay-Dale; PartNumber (none) -> CRCW0402102KFKED
- R13: renamed from R17; value 47k -> 4.99k; footprint Resistor_SMD:R_0805_2012Metric_Pad1.20x1.40mm_HandSolder -> Resistor_SMD:R_0402_1005Metric; LCSC (none) -> C482195; Manufacturer (none) -> Vishay-Dale; PartNumber (none) -> CRCW04024K99FKED
- R14: renamed from R18; value 47k -> 4.99k; footprint Resistor_SMD:R_0805_2012Metric_Pad1.20x1.40mm_HandSolder -> Resistor_SMD:R_0402_1005Metric; LCSC (none) -> C482195; Manufacturer (none) -> Vishay-Dale; PartNumber (none) -> CRCW04024K99FKED
- R15: value 15k -> 102k; footprint Resistor_SMD:R_0805_2012Metric_Pad1.20x1.40mm_HandSolder -> Resistor_SMD:R_0402_1005Metric; LCSC (none) -> C481920; Manufacturer (none) -> Vishay-Dale; PartNumber (none) -> CRCW0402102KFKED
- R17: renamed from R21; value 47k -> 49.9k; footprint Resistor_SMD:R_0805_2012Metric_Pad1.20x1.40mm_HandSolder -> Resistor_SMD:R_0402_1005Metric; LCSC (none) -> C350874; Manufacturer (none) -> Vishay-Dale; PartNumber (none) -> CRCW040249K9FKED
- R18: renamed from R22; value 15k -> 12.7k; footprint Resistor_SMD:R_0805_2012Metric_Pad1.20x1.40mm_HandSolder -> Resistor_SMD:R_0402_1005Metric; LCSC (none) -> C481941; Manufacturer (none) -> Vishay-Dale; PartNumber (none) -> CRCW040212K7FKED
- R21: renamed from R25; value 100k -> 49.9k; footprint Resistor_SMD:R_0805_2012Metric_Pad1.20x1.40mm_HandSolder -> Resistor_SMD:R_0402_1005Metric; LCSC (none) -> C350874; Manufacturer (none) -> Vishay-Dale; PartNumber (none) -> CRCW040249K9FKED
- R22: renamed from R26; footprint Resistor_SMD:R_1210_3225Metric_Pad1.30x2.65mm_HandSolder -> Resistor_SMD:R_0402_1005Metric; LCSC (none) -> C482122; Manufacturer (none) -> Vishay-Dale; PartNumber (none) -> CRCW040227R0FKED
- R3: value 5.6k -> 11.3k; footprint Resistor_SMD:R_1206_3216Metric_Pad1.30x1.75mm_HandSolder -> Resistor_SMD:R_0402_1005Metric; LCSC (none) -> C481933; Manufacturer (none) -> Vishay-Dale; PartNumber (none) -> CRCW040211K3FKED
- R4: value 47k -> 49.9k; footprint Resistor_SMD:R_0805_2012Metric_Pad1.20x1.40mm_HandSolder -> Resistor_SMD:R_0402_1005Metric; LCSC (none) -> C350874; Manufacturer (none) -> Vishay-Dale; PartNumber (none) -> CRCW040249K9FKED
- R5: value 120k -> 150k; footprint Resistor_SMD:R_0805_2012Metric_Pad1.20x1.40mm_HandSolder -> Resistor_SMD:R_0402_1005Metric; LCSC (none) -> C328301; Manufacturer (none) -> RESI; PartNumber (none) -> AECR0402F150KK9
- R6: renamed from R8; footprint Resistor_SMD:R_0805_2012Metric_Pad1.20x1.40mm_HandSolder -> Resistor_SMD:R_0402_1005Metric; LCSC (none) -> C481926; Manufacturer (none) -> Vishay-Dale; PartNumber (none) -> CRCW040210R0FKED
- R7: renamed from R9; footprint Resistor_SMD:R_0805_2012Metric_Pad1.20x1.40mm_HandSolder -> Resistor_SMD:R_0402_1005Metric; LCSC (none) -> C191587; Manufacturer (none) -> Vishay-Dale; PartNumber (none) -> CRCW040215K0FKED
- R9: renamed from R11; footprint Resistor_SMD:R_1206_3216Metric_Pad1.30x1.75mm_HandSolder -> Resistor_SMD:R_1206_3216Metric; LCSC (none) -> C5629523; Manufacturer (none) -> Bourns; PartNumber (none) -> CRF1206-FZ-R010ELF
- TP1, TP2: LCSC (none) -> C238131; PartNumber (none) -> 5019
- TP11: renamed from TP10; LCSC (none) -> C238131; PartNumber (none) -> 5019
- TP4: renamed from TP3; LCSC (none) -> C238131; PartNumber (none) -> 5019
- TP7: renamed from TP6; LCSC (none) -> C238131; PartNumber (none) -> 5019
- TP8: renamed from TP7; LCSC (none) -> C238131; PartNumber (none) -> 5019
- TP9: renamed from TP8; LCSC (none) -> C238131; PartNumber (none) -> 5019
- U1: LCSC (none) -> C42116949; Manufacturer (none) -> Texas Instruments; PartNumber (none) -> TPS551892QWRYQRQ1
- U2: LCSC (none) -> C6253250; Manufacturer (none) -> TDK; PartNumber (none) -> FS1403-5000-AL
Connections:
- net 12V_IN is gone; now on net V_BAT+: C29.1, C30.1, R22.1, U2.12 (PVIN), U2.13 (PVIN), U2.14 (PVIN), U2.17 (PVIN)
- net *CC_12: now also C25.2, R15.1; no longer C25.1
- net +12V: now also C10.1, C11.1, C12.1, C13.1, C14.1, C15.1, C9.1, R9.2, U1.11 (VOUT), R8.1; no longer R12.1, R21.1
- net EN_12: now also C24.2; no longer C24.1
- net EN_5: now also C28.2; no longer C28.1
- net GND: now also C23.1, C24.1, C25.1, C28.1, R18.2, R3.1, R4.2, C33.2, C34.1, C35.2, R16.1; no longer C23.2, C24.2, C25.2, C28.2
- net PG_12: now also C23.2, R12.1; no longer C23.1, R12.2
- net VCC_12: now also R12.2, R15.2
- net V_BAT+: now also R17.1, C33.1, C34.2
- net at R10.2: now also J3.1 (Pin_1), R11.1
- net at R2.2, R3.2, U1.14 (FB): now also TP3.1
- net at U2.6 (ADDR): now also R16.2
- net VCC_5: now reaches C32.1, U2.10 (VCC)
- net VCC_5: now also R21.1
- net at R22.2, TP11.1, U2.11 (VIN): now also C35.1
- net at C6.2, U1.13 (ISN): now also R6.2
- net at C6.1, U1.12 (ISP): now also R8.2; no longer R6.2
- net DITH/SYNC: now reaches C1.2, U1.5 (DITH/SYNC)
Other:
- moved on the sheet: C1, C2, C26, C27, C29, C30, C31, C32, C9, J10, J3, J7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
