File: PowerPCB/PowerPCB.kicad_pcb (KiCad board)
At the start: 4 copper layers, 100 x 60 mm, 81 parts, among them J1 Battery, J10 Conn_01x02, J2 Conn_01x02, J3 12Vout, J4 Conn_01x03, J5 5Vout, J6 Conn_01x03, J7 Conn_01x03, J8 Conn_01x02, J9 Conn_01x03, U1 TPS551892QWRYQRQ1, U2 FS1403-5000-AL

Commit message: placa conectada
Parts:
- moved R26 104.0 mm to (169.5, 76.5), turned to -90 degrees
- moved U2 91.3 mm to (178.0, 85.5), turned to 180 degrees
- moved TP9 84.6 mm to (166.5, 87.0)
- moved TP10 83.9 mm to (169.6, 82.5)
- moved C30 81.2 mm to (171.5, 90.0), turned to -90 degrees
- moved C32 74.3 mm to (169.5, 71.5), turned to 180 degrees
- moved J6 69.0 mm to (162.0, 74.5), turned to 180 degrees
- moved C29 68.2 mm to (174.5, 90.0), turned to -90 degrees
- moved J9 65.0 mm to (177.5, 69.0), turned to 90 degrees
- moved TP8 64.8 mm to (187.5, 81.5)
- moved R24 61.8 mm to (176.5, 77.0)
- moved J5 61.6 mm to (204.5, 77.0)
- moved J10 61.6 mm to (204.0, 98.5)
- moved R20 56.4 mm to (169.5, 68.5)
- moved C31 56.2 mm to (187.0, 90.0), turned to -90 degrees
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Routing:
- net V_BAT+: track 38.1 -> 124.8 mm, vias 16 -> 22
- net V_OUT_12+: track 144.9 -> 227.6 mm, vias 3 -> 7
- net V_OUT_5+: track 0.00 -> 41.9 mm, vias 0 -> 4
- net 12V_IN: track 0.00 -> 37.8 mm, vias 0 -> 5
- net SDA: track 0.00 -> 33.5 mm
- net PG_5: track 0.00 -> 31.3 mm, vias 0 -> 2
- net VBUS: track 0.00 -> 29.5 mm, vias 0 -> 2
- net SCL: track 0.00 -> 27.5 mm
- net EN_5: track 0.00 -> 23.7 mm, vias 0 -> 4
- net Net-(U2-VCC): track 0.00 -> 16.5 mm
- net Net-(U2-VIN): track 0.00 -> 14.1 mm
- net Net-(R20-Pad2): track 0.00 -> 9.62 mm
- net Net-(J9-Pin_1): track 0.00 -> 9.52 mm
- net Net-(U2-ADDR): track 0.00 -> 7.89 mm
- net Net-(R22-Pad2): track 0.00 -> 3.00 mm
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Other:
- board text added: "${REFERENCE}"

Commit message: PCB finished
Parts:
- moved C31 7.71 mm to (179.4, 89.0), turned to 180 degrees
- moved R25 4.90 mm to (179.4, 91.5), turned to 0 degrees
- moved C26 3.40 mm to (198.0, 75.9)
- moved C27 3.40 mm to (200.5, 75.9)
- turned C32 to 0 degrees
Routing:
- net V_OUT_12+: track 227.6 -> 202.2 mm, vias 7 -> 3
- net V_OUT_5+: track 41.9 -> 29.3 mm, vias 4 -> 0
- net 12V_IN: track 37.8 -> 35.8 mm, vias 5 -> 0
- net PG_5: track 31.3 -> 33.3 mm, vias 2 -> 1
- net Net-(U2-ADDR): track 7.89 -> 9.79 mm, vias 0 -> 2
- net SDA: track 33.5 -> 35.3 mm
- net VCC_12: track 34.0 -> 32.3 mm, vias 3 -> 2
- net Net-(U2-VCC): track 16.5 -> 17.4 mm
- net V_BAT+: track 124.8 -> 124.7 mm, vias 22 -> 0
- net V_BAT-: vias 24 -> 52
- net Net-(U1A-VOUT): vias 7 -> 2
- added copper zone on F.Cu, net 12V_IN
- added copper zone on F.Cu, net V_OUT_5+

Commit message: minor fixes
Parts:
- J1, J3: footprint TerminalBlock_4Ucon:TerminalBlock_4Ucon_1x02_P3.50mm_Horizontal -> TerminalBlock_MetzConnect:TerminalBlock_MetzConnect_Type094_RT03502HBLU_1x02_P5.00mm_Horizontal
- J5: footprint Connector_PinHeader_2.54mm:PinHeader_1x02_P2.54mm_Vertical -> TerminalBlock_MetzConnect:TerminalBlock_MetzConnect_Type094_RT03502HBLU_1x02_P5.00mm_Horizontal
- moved C27 3.90 mm to (196.6, 76.0)
- moved C26 3.80 mm to (194.2, 76.0)
- moved J5 1.97 mm to (203.2, 78.5), turned to 90 degrees
- moved TP7 1.66 mm to (114.2, 123.8)
- moved C28 0.30 mm to (187.2, 78.0)
- moved R23 0.20 mm to (187.8, 74.0)
Routing:
- net SCL: track 27.5 -> 34.2 mm
- net V_BAT-: track 113.2 -> 107.5 mm
- net VBUS: track 29.5 -> 33.5 mm, vias 2 -> 0
- net VCC_12: track 32.3 -> 36.1 mm, vias 2 -> 3
- net V_OUT_5+: track 29.3 -> 28.6 mm

Commit message: minor changes
Parts:
- moved TP5 54.4 mm to (193.6, 121.4), turned to -90 degrees
- moved TP7 0.28 mm to (114.4, 123.6)
Routing:
- net V_BAT-: track 107.5 -> 121.5 mm
Changed lines of the file:
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@@
 		(tags "capacitor handsolder")
 		(property "Reference" "C30"
-			(at 0 -1.68 90)
+			(at 0 -1.5 90)
 			(layer "F.SilkS")
 			(effects
@@
 		(tags "capacitor handsolder")
 		(property "Reference" "C28"
-			(at 0 0 0)
+			(at 0 -1.8 0)
 			(layer "F.SilkS")
 			(effects
@@
 		)
 		(property "Value" "0.1uF"
-			(at 0 1.85 0)
+			(at 4.2 0 0)
 			(layer "F.Fab")
 			(effects
@@
 		)
 		(property "Value" "100k"
-			(at 0 1.65 0)
+			(at -7 -0.066667 0)
 			(layer "F.Fab")
 			(effects
@@
 		(tags "capacitor handsolder")
 		(property "Reference" "C27"
-			(at 0 1.6 270)
+			(at 2.6 0 0)
 			(layer "F.SilkS")
 			(effects
@@
 		)
 		(property "Value" "47k"
-			(at 0 1.65 0)
+			(at 1.544669 0.6 0)
 			(layer "F.Fab")
 			(effects
@@
 	(footprint "TestPoint:TestPoint_Keystone_5019_Miniature"
 		(layer "F.Cu")
-		(at 114.2 123.8)
+		(at 114.4 123.6)
 		(descr "Keystone SMT Miniature Test Point 5019, http://www.keyelco.com/product-pdf.cfm?p=1357")
 		(tags "Test Point")
@@
 		(tags "resistor handsolder")
 		(property "Reference" "R25"
-			(at 0 1.754513 0)
+			(at 3.4498 0.1 0)
 			(layer "F.SilkS")
 			(effects
@@
 		)
 		(property "Value" "15k"
-			(at 0 1.65 0)
+			(at 6.6 0 0)
 			(layer "F.Fab")
 			(effects
@@
 		)
 		(property "Value" "100k"
-			(at 0 1.65 0)
+			(at 7 0.066667 0)
 			(layer "F.Fab")
 			(effects
@@
 		(tags "capacitor handsolder")
 		(property "Reference" "C31"
-			(at 0 -1.68 0)
+			(at -3.2498 0.034663 0)
 			(layer "F.SilkS")
 			(effects
@@
 		)
 		(property "Value" "0.01uF"
-			(at 0 1.68 0)
+			(at -2.2498 1.434663 0)
 			(layer "F.Fab")
 			(effects
@@
 		)
 		(property "Value" "47k"
-			(at 0 1.65 0)
+			(at -6.6 0.066666 0)
 			(layer "F.Fab")
 			(effects
@@
 		(tags "resistor handsolder")
 		(property "Reference" "R24"
-			(at 0 -1.65 0)
+			(at 0 -1.4 0)
 			(layer "F.SilkS")
 			(effects
@@
 		(tags "capacitor handsolder")
 		(property "Reference" "C26"
-			(at 0 -1.6 270)
+			(at 2.6 -0.4 0)
 			(layer "F.SilkS")
 			(effects
@@
 	(footprint "TestPoint:TestPoint_Keystone_5019_Miniature"
 		(layer "F.Cu")
-		(at 139.2 121.6 180)
+		(at 193.6 121.4 -90)
 		(descr "Keystone SMT Miniature Test Point 5019, http://www.keyelco.com/product-pdf.cfm?p=1357")
 		(tags "Test Point")
 		(property "Reference" "TP5"
-			(at 0 -2.4 180)
+			(at 0 -2.4 90)
 			(layer "F.SilkS")
 			(effects
@@
 		)
 		(property "Value" "TestPoint"
-			(at 0 2.25 0)
+			(at 0 2.25 90)
 			(layer "F.Fab")
 			(effects
@@
 		)
 		(property "Datasheet" "~"
-			(at 0.02 -2.81 180)
+			(at 0.02 -2.81 270)
 			(unlocked yes)
 			(layer "F.Fab")
@@
 		)
 		(property "Description" "test point"
-			(at 0.02 -2.81 180)
+			(at 0.02 -2.81 270)
 			(unlocked yes)
 			(layer "F.Fab")
@@
 		)
 		(fp_line
-			(start 2.35 1.45)
-			(end -2.35 1.45)
+			(start -2.35 1.45)
+			(end -2.35 -1.45)
 			(stroke
 				(width 0.05)
@@
 		)
 		(fp_line
-			(start 2.35 -1.45)
-			(end 2.35 1.45)
+			(start 2.35 1.45)
+			(end -2.35 1.45)
 			(stroke
 				(width 0.05)
@@
 		)
 		(fp_line
-			(start -2.35 1.45)
-			(end -2.35 -1.45)
+			(start -2.35 -1.45)
+			(end 2.35 -1.45)
 			(stroke
 				(width 0.05)
@@
 		)
 		(fp_line
-			(start -2.35 -1.45)
-			(end 2.35 -1.45)
+			(start 2.35 -1.45)
+			(end 2.35 1.45)
 			(stroke
 				(width 0.05)
@@
 		)
 		(fp_rect
-			(start 0 0.5)
-			(end 1.25 1)
+			(start -1.25 0.5)
+			(end 0 1)
 			(stroke
 				(width 0.1)
@@
 		)
 		(fp_rect
-			(start 0 -1)
-			(end 1.25 -0.5)
+			(start 0 0.5)
+			(end 1.25 1)
 			(stroke
 				(width 0.1)
@@
 		)
 		(fp_rect
-			(start -1.25 0.5)
-			(end 0 1)
+			(start -1.9 -0.5)
+			(end 1.9 0.5)
 			(stroke
 				(width 0.1)
@@
 		)
 		(fp_rect
-			(start -1.9 -0.5)
-			(end 1.9 0.5)
+			(start 0 -1)
+			(end 1.25 -0.5)
 			(stroke
 				(width 0.1)
@@
 		)
 		(fp_text user "${REFERENCE}"
-			(at 0 0 0)
+			(at 0 0 90)
 			(layer "F.Fab")
 			(effects
@@
 		)
 		(pad "1" smd roundrect
-			(at 0 0 180)
+			(at 0 0 270)
 			(size 3.8 2)
 			(layers "F.Cu" "F.Mask" "F.Paste")
@@
 		)
 		(property "Value" "100k"
-			(at 0 1.65 90)
+			(at -0.2 -2.8 180)
 			(layer "F.Fab")
 			(effects
@@
 		(tags "Test Point")
 		(property "Reference" "TP8"
-			(at 0 -2.25 0)
+			(at 3.5 1.3 0)
 			(layer "F.SilkS")
 			(effects
@@
 		)
 		(property "Value" "22uF"
-			(at 0 1.68 90)
+			(at 0 1.5 90)
 			(layer "F.Fab")
 			(effects
@@
 		)
 		(property "Value" "0.01uF"
-			(at 0 1.68 90)
+			(at 2.6 -3.8 180)
 			(layer "F.Fab")
 			(effects
@@
 		(tags "resistor handsolder")
 		(property "Reference" "R17"
-			(at -1.01875 -3.66875 90)
+			(at -0.2 -1.8 90)
 			(layer "F.SilkS")
 			(effects
@@
 		)
 		(property "Value" "47k"
-			(at 0 1.65 90)
+			(at -2.6 0 180)
 			(layer "F.Fab")
 			(effects
@@
 	)
 	(segment
+		(start 114.4 123.6)
+		(end 114.4 118.6)
+		(width 1.4)
+		(layer "F.Cu")
+		(net 2)
+	)
+	(segment
 		(start 139.2 121.6)
 		(end 149.8 121.6)
@@
 	)
 	(segment
+		(start 193.6 121.4)
+		(end 202.6 121.4)
+		(width 1.4)
+		(layer "F.Cu")
+		(net 2)
+	)
+	(segment
 		(start 114.4 118.6)
 		(end 136.2 118.6)
@@
 	)
 	(zone
+		(net 2)
+		(net_name "V_BAT-")
+		(layer "F.Cu")
+		(name "$teardrop_padvia$")
+		(hatch none 0.1)
+		(priority 30000)
+		(attr
+			(teardrop
+				(type padvia)
+			)
+		)
+		(connect_pads yes
+			(clearance 0)
+		)
+		(min_thickness 0.0254)
+		(filled_areas_thickness no)
+		(fill yes
+			(thermal_gap 0.5)
+			(thermal_bridge_width 0.5)
+			(island_removal_mode 1)
+			(island_area_min 10)
+		)
+		(polygon
+			(pts
+				(xy 115.1 121.6) (xy 113.7 121.6) (xy 113.4 122.6) (xy 114.4 123.601) (xy 115.4 122.6)
+			)
+		)
+	)
+	(zone
 		(net 17)
 		(net_name "PG_12")
@@
 	)
 	(zone
+		(net 2)
+		(net_name "V_BAT-")
+		(layer "F.Cu")
+		(name "$teardrop_padvia$")
+		(hatch none 0.1)
+		(priority 30000)
+		(attr
+			(teardrop
+				(type padvia)
+			)
+		)
+		(connect_pads yes
+			(clearance 0)
+		)
+		(min_thickness 0.0254)
+		(filled_areas_thickness no)
+		(fill yes
+			(thermal_gap 0.5)
+			(thermal_bridge_width 0.5)
+			(island_removal_mode 1)
+			(island_area_min 10)
+		)
+		(polygon
+			(pts
+				(xy 195.6 122.1) (xy 195.6 120.7) (xy 194.6 120.4) (xy 193.599 121.4) (xy 194.6 122.4)
+			)
+		)
+	)
+	(zone
 		(net 12)
 		(net_name "Net-(U1A-COMP)")
@@
 	)
 	(zone
-		(net 2)
-		(net_name "V_BAT-")
-		(layer "F.Cu")
-		(name "$teardrop_padvia$")
-		(hatch none 0.1)
-		(priority 30003)
-		(attr
-			(teardrop
-				(type padvia)
-			)
-		)
-		(connect_pads yes
-			(clearance 0)
-		)
-		(min_thickness 0.0254)
-		(filled_areas_thickness no)
-		(fill yes
-			(thermal_gap 0.5)
-			(thermal_bridge_width 0.5)
-			(island_removal_mode 1)
-			(island_area_min 10)
-		)
-		(polygon
-			(pts
-				(xy 137.846447 119.53934) (xy 137.13934 120.246447) (xy 137.3 121.114214) (xy 139.200707 121.600707)
-				(xy 139.614214 120.6)
-			)
-		)
-	)
-	(zone
 		(net 38)
 		(net_name "Net-(U2-ADDR)")
@@
 			)
 		)
-	)
-	(zone
-		(net 2)
-		(net_name "V_BAT-")
-		(layer "F.Cu")
-		(name "$teardrop_padvia$")
-		(hatch none 0.1)
-		(priority 30002)
-		(attr
-			(teardrop
-				(type padvia)
-			)
-		)
-		(connect_pads yes
-			(clearance 0)
-		)
-		(min_thickness 0.0254)
-		(filled_areas_thickness no)
-		(fill yes
-			(thermal_gap 0.5)
-			(thermal_bridge_width 0.5)
-			(island_removal_mode 1)
-			(island_area_min 10)
-		)
-		(polygon
-			(pts
-				(xy 142.1 122.1) (xy 142.1 121.1) (xy 140.945671 120.61903) (xy 139.199 121.6) (xy 140.945671 122.58097)
-			)
-		)

Commit message: PowerPCB v2
Parts:
- removed J6: Conn_01x03, Connector_PinHeader_2.54mm:PinHeader_1x03_P2.54mm_Vertical
- removed the R10 at (158.4, 101.3)
- removed the R14 at (117.2, 97.5)
- removed R19, R20, R23: 100k, Resistor_SMD:R_0805_2012Metric_Pad1.20x1.40mm_HandSolder
- removed R24: 0, Resistor_SMD:R_0805_2012Metric_Pad1.20x1.40mm_HandSolder
- removed the R6 at (157.8, 86.2)
- removed the R7 at (134.0, 91.3)
- removed the TP4 at (191.0, 111.4)
- removed TP5: TestPoint, TestPoint:TestPoint_Keystone_5019_Miniature
- removed the TP9 at (166.5, 87.0)
- added C33: 68uF, Capacitor_SMD:CP_Elec_8x10, F.Cu at (122.7, 101.2)
- added C34: 0.1uF, Capacitor_SMD:C_0402_1005Metric, F.Cu at (128.3, 92.1)
- added C35: 1uF, Capacitor_SMD:C_0603_1608Metric, F.Cu at (123.4, 86.4)
- added R16: 0, Resistor_SMD:R_0402_1005Metric, F.Cu at (131.5, 88.2)
- added R8: 10, Resistor_SMD:R_0402_1005Metric, F.Cu at (154.4, 94.7)
- added TP3: TestPoint, TestPoint:TestPoint_Keystone_5019_Miniature, F.Cu at (166.6, 122.5)
- C1, C23, C25, C31, C7: footprint Capacitor_SMD:C_0805_2012Metric_Pad1.18x1.45mm_HandSolder -> Capacitor_SMD:C_0402_1005Metric
- C10, C11, C12, C18, C19, C26, C27, C29, C30, C32: footprint Capacitor_SMD:C_0805_2012Metric_Pad1.18x1.45mm_HandSolder -> Capacitor_SMD:C_1206_3216Metric
- C13, C16, C20, C3, C4, C5: footprint Capacitor_SMD:C_1206_3216Metric_Pad1.33x1.80mm_HandSolder -> Capacitor_SMD:C_0603_1608Metric
- C14, C21: footprint Capacitor_SMD:C_1206_3216Metric_Pad1.33x1.80mm_HandSolder -> Capacitor_SMD:C_0402_1005Metric; moved to B.Cu
- C15, C2, C22, C24, C28, C6, C8: footprint Capacitor_SMD:C_1206_3216Metric_Pad1.33x1.80mm_HandSolder -> Capacitor_SMD:C_0402_1005Metric
- C9: footprint Capacitor_SMD:CP_Elec_6.3x5.4 -> Capacitor_SMD:CP_Elec_6.3x5.8
- R1: value 51 -> 49.9; footprint Resistor_SMD:R_0805_2012Metric_Pad1.20x1.40mm_HandSolder -> Resistor_SMD:R_0402_1005Metric
- R10: renamed from R13; value 100k -> 147k; footprint Resistor_SMD:R_0805_2012Metric_Pad1.20x1.40mm_HandSolder -> Resistor_SMD:R_0402_1005Metric
- R11: renamed from R16; value 100k -> 115k; footprint Resistor_SMD:R_0805_2012Metric_Pad1.20x1.40mm_HandSolder -> Resistor_SMD:R_0402_1005Metric
- R12, R2: value 100k -> 102k; footprint Resistor_SMD:R_0805_2012Metric_Pad1.20x1.40mm_HandSolder -> Resistor_SMD:R_0402_1005Metric
- R13: renamed from R17; value 47k -> 4.99k; footprint Resistor_SMD:R_0805_2012Metric_Pad1.20x1.40mm_HandSolder -> Resistor_SMD:R_0402_1005Metric
- R14: renamed from R18; value 47k -> 4.99k; footprint Resistor_SMD:R_0805_2012Metric_Pad1.20x1.40mm_HandSolder -> Resistor_SMD:R_0402_1005Metric
- R15: value 15k -> 102k; footprint Resistor_SMD:R_0805_2012Metric_Pad1.20x1.40mm_HandSolder -> Resistor_SMD:R_0402_1005Metric
- R17: renamed from R21; value 47k -> 49.9k; footprint Resistor_SMD:R_0805_2012Metric_Pad1.20x1.40mm_HandSolder -> Resistor_SMD:R_0402_1005Metric
- R18: renamed from R22; value 15k -> 12.7k; footprint Resistor_SMD:R_0805_2012Metric_Pad1.20x1.40mm_HandSolder -> Resistor_SMD:R_0402_1005Metric
- R21: renamed from R25; value 100k -> 49.9k; footprint Resistor_SMD:R_0805_2012Metric_Pad1.20x1.40mm_HandSolder -> Resistor_SMD:R_0402_1005Metric
- R22: renamed from R26; footprint Resistor_SMD:R_1210_3225Metric_Pad1.30x2.65mm_HandSolder -> Resistor_SMD:R_0402_1005Metric
- R3: value 5.6k -> 11.3k; footprint Resistor_SMD:R_1206_3216Metric_Pad1.30x1.75mm_HandSolder -> Resistor_SMD:R_0402_1005Metric
- R4: value 47k -> 49.9k; footprint Resistor_SMD:R_0805_2012Metric_Pad1.20x1.40mm_HandSolder -> Resistor_SMD:R_0402_1005Metric
- R5: value 120k -> 150k; footprint Resistor_SMD:R_0805_2012Metric_Pad1.20x1.40mm_HandSolder -> Resistor_SMD:R_0402_1005Metric
- R6: renamed from R8; footprint Resistor_SMD:R_0805_2012Metric_Pad1.20x1.40mm_HandSolder -> Resistor_SMD:R_0402_1005Metric
- R7: renamed from R9; footprint Resistor_SMD:R_0805_2012Metric_Pad1.20x1.40mm_HandSolder -> Resistor_SMD:R_0402_1005Metric
- R9: renamed from R11; footprint Resistor_SMD:R_1206_3216Metric_Pad1.30x1.75mm_HandSolder -> Resistor_SMD:R_1206_3216Metric
- moved C28 79.0 mm to (119.1, 118.0)
- moved J9 76.2 mm to (122.0, 121.3), turned to -90 degrees
- moved R18 75.3 mm to (122.6, 118.9)
- moved J10 72.4 mm to (135.3, 121.3), turned to -90 degrees
- moved R17 69.5 mm to (122.6, 117.9), turned to 180 degrees
- moved J7 66.6 mm to (147.0, 121.3), turned to -90 degrees
- moved R21 53.2 mm to (133.4, 118.3)
- moved C31 52.6 mm to (135.7, 118.3), turned to 0 degrees
- moved R13 52.5 mm to (144.9, 118.6), turned to 180 degrees
- moved J8 51.6 mm to (145.7, 113.6), turned to -90 degrees
- moved U2 50.4 mm to (127.8, 89.6)
- moved R14 50.3 mm to (142.4, 118.6)
- moved R22 48.7 mm to (122.1, 87.8), turned to 0 degrees
- moved C32 47.1 mm to (124.2, 84.3)
- moved C25 44.6 mm to (143.6, 110.6), turned to 0 degrees
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- renumbered J4 to J3, J3 to J4, TP10 to TP11, TP3 to TP4, TP6 to TP7, TP7 to TP8, TP8 to TP9
Connections:
- net Net-(U1A-DITH/SYNC) renamed /DITH/SYNC
- C1 pad 1: V_BAT- -> GND
- C10 pad 1: Net-(U1A-VOUT) -> V_OUT_12+
- C10 pad 2: V_BAT- -> GND
- C11 pad 1: Net-(U1A-VOUT) -> V_OUT_12+
- C11 pad 2: V_BAT- -> GND
- C12 pad 1: Net-(U1A-VOUT) -> V_OUT_12+
- C12 pad 2: V_BAT- -> GND
- C13 pad 1: Net-(U1A-VOUT) -> V_OUT_12+
- C13 pad 2: V_BAT- -> GND
- C14 pad 1: Net-(U1A-VOUT) -> V_OUT_12+
- C14 pad 2: V_BAT- -> GND
- C15 pad 1: Net-(U1A-VOUT) -> V_OUT_12+
- C15 pad 2: V_BAT- -> GND
- C16 pad 2: V_BAT- -> GND
- C17 pad 2: V_BAT- -> GND
- C18 pad 2: V_BAT- -> GND
- C19 pad 2: V_BAT- -> GND
- C2 pad 1: V_BAT- -> GND
- C20 pad 2: V_BAT- -> GND
- C21 pad 2: V_BAT- -> GND
- C22 pad 2: V_BAT- -> GND
- C23 pad 1: PG_12 -> GND
- C23 pad 2: V_BAT- -> PG_12
- C24 pad 1: EN_12 -> GND
- C24 pad 2: V_BAT- -> EN_12
- C25 pad 1: *CC_12 -> GND
- C25 pad 2: V_BAT- -> *CC_12
- C26 pad 2: V_BAT- -> GND
- C27 pad 2: V_BAT- -> GND
- C28 pad 1: EN_5 -> GND
- C28 pad 2: V_BAT- -> EN_5
- C29 pad 1: 12V_IN -> V_BAT+
- C29 pad 2: V_BAT- -> GND
- C30 pad 1: 12V_IN -> V_BAT+
- C30 pad 2: V_BAT- -> GND
- C31 pad 2: V_BAT- -> GND
- C32 pad 1: Net-(U2-VCC) -> /VCC_5
- C32 pad 2: V_BAT- -> GND
- C5 pad 2: V_BAT- -> GND
- C7 pad 2: V_BAT- -> GND
- C8 pad 2: V_BAT- -> GND
- C9 pad 1: Net-(U1A-VOUT) -> V_OUT_12+
- C9 pad 2: V_BAT- -> GND
- J1 pad 2: V_BAT- -> GND
- J10 pad 2: V_BAT- -> GND
- J2 pad 2: V_BAT- -> GND
- J3 pad 1: Net-(J4-Pin_1) -> Net-(J3-Pin_1)
- J3 pad 3: V_BAT- -> GND
- J4 pad 2: V_BAT- -> GND
- J5 pad 2: V_BAT- -> GND
- J8 pad 2: V_BAT- -> GND
- J9 pad 3: V_BAT- -> GND
- R10 pad 2: Net-(R13-Pad2) -> Net-(J3-Pin_1)
- R11 pad 1: Net-(R15-Pad2) -> Net-(J3-Pin_1)
- R11 pad 2: V_BAT- -> GND
- R12 pad 1: V_OUT_12+ -> PG_12
- R12 pad 2: PG_12 -> VCC_12
- R15 pad 1: Net-(J4-Pin_1) -> *CC_12
- R15 pad 2: Net-(R15-Pad2) -> VCC_12
- R17 pad 1: Net-(R20-Pad2) -> V_BAT+
- R18 pad 2: Net-(R22-Pad2) -> GND
- R21 pad 1: V_OUT_12+ -> /VCC_5
- R22 pad 1: 12V_IN -> V_BAT+
- R3 pad 1: Net-(R3-Pad1) -> GND
- R4 pad 2: Net-(R4-Pad2) -> GND
- R5 pad 2: V_BAT- -> GND
- R6 pad 2: Net-(U1A-ISP) -> Net-(U1A-ISN)
- R9 pad 2: Net-(U1A-VOUT) -> V_OUT_12+
- TP8 pad 1: V_BAT- -> GND
- U1 pad 11: Net-(U1A-VOUT) -> V_OUT_12+
- U1 pad 17: V_BAT- -> GND
- U1 pad 9: V_BAT- -> GND
- U2 pad 10: Net-(U2-VCC) -> /VCC_5
- U2 pad 12: 12V_IN -> V_BAT+
- U2 pad 13: 12V_IN -> V_BAT+
- U2 pad 14: 12V_IN -> V_BAT+
- U2 pad 16: V_BAT- -> GND
- U2 pad 17: 12V_IN -> V_BAT+
- U2 pad 8: V_BAT- -> GND
- U2 pad 9: V_BAT- -> GND
Routing:
- net V_OUT_12+: track 202.2 -> 57.0 mm, vias 3 -> 55
- net V_BAT-: track 121.5 -> 0.00 mm, vias 52 -> 0
- net V_BAT+: track 124.7 -> 45.2 mm, vias 0 -> 47
- net /VCC_5: track 0.00 -> 71.7 mm, vias 0 -> 2
- net Net-(U2-VIN): track 14.0 -> 71.1 mm, vias 0 -> 2
- net Net-(R1-Pad2): track 9.85 -> 51.1 mm, vias 0 -> 3
- net Net-(U1A-FB): track 14.4 -> 50.9 mm, vias 0 -> 2
- net 12V_IN: track 35.8 -> 0.00 mm
- net VBUS: track 33.5 -> 6.36 mm
- net V_OUT_5+: track 28.6 -> 3.18 mm, vias 0 -> 62
- net EN_5: track 23.4 -> 47.9 mm, vias 4 -> 1
- net PG_5: track 33.2 -> 57.0 mm
- net Net-(U2-VCC): track 17.4 -> 0.00 mm
- net VCC_12: track 36.1 -> 52.6 mm, vias 3 -> 4
- net Net-(U1A-VOUT): track 11.5 -> 0.00 mm, vias 2 -> 0
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- added copper zone on B.Cu, net GND
- added copper zone on F.Cu, net GND
- added copper zone on In2.Cu, net GND
- added copper zone on F.Cu, net VCC_12
- added copper zone on B.Cu, net V_BAT+
- added copper zone on B.Cu, net V_OUT_12+
- added copper zone on F.Cu, net V_OUT_12+
- added copper zone on B.Cu, net V_OUT_5+
- removed copper zone on F.Cu, net 12V_IN
- removed copper zone on F.Cu, net Net-(U1A-VOUT)
- removed copper zone on B.Cu, net V_BAT-
- removed copper zone on F.Cu, net V_BAT-
Other:
- board size 100 x 60 mm -> 82.3 x 55.3 mm
- board text added: "CC_12"
- board text added: "EN_12"
- board text added: "EN_5"
- board text added: "OFF"
- board text added: "ON"
- board text added: "PG_12"
- board text added: "PG_5"
- board text added: "SCL"
- board text added: "SDA"
- board text added: "VBUS"
- board text removed: "${REFERENCE}"

Commit message: Final PCB revision
Parts:
- added G***: LOGO, LOGO, F.Cu at (175.0, 81.4)
- OUT 12V: renamed from TP2
- OUT 5V: renamed from TP9
- U1 FB: renamed from TP3
- U2 VIN: renamed from TP11
- moved C17 3.10 mm to (135.6, 101.4)
- moved C33 3.10 mm to (125.8, 101.4)
- moved J1 0.70 mm to (113.0, 97.8)
- renumbered TP8 to GND, TP7 to VBAT
Routing:
- net V_OUT_5+: vias 62 -> 65
- net V_BAT+: vias 47 -> 49
