File: LogicPCB/LogicPCB.kicad_sch (KiCad schematic)
At the start: 70 parts, among them IC1 DRV8411PWPR, IC2 DRV8411PWPR, IC3 DRV8411PWPR, J1 POWER_IN, J3 DC_OUT, J4 ICSP, J5 RS232, SW1 SW_Push_Dual, U1 DRV8871DDA, U2 ATmega2560-16A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

Commit message: LogicPCB done
Parts:
- removed D1: 1N5819, Diode_THT:D_DO-41_SOD81_P10.16mm_Horizontal, symbol Diode:1N5819
- removed TP3: TestPoint, TestPoint:TestPoint_Pad_D1.0mm, symbol Connector:TestPoint
Connections:
- net FAULT_STP23 is gone; now on net FAULT_STP3: IC3.8 (FAULT_N), R10.1
- net FAULT_STP1: now also U2.54 (PC1); no longer U2.53 (PC0)
- net FAULT_STP2: now also U2.56 (PC3); no longer U2.54 (PC1)
- net FAULT_STP3: now also U2.58 (PC5); no longer U2.55 (PC2)
- net OUT1_DC: now also J3.2; no longer J3.1
- net OUT2_DC: now also J3.1; no longer J3.2
- net SLEEP_STP1: now also U2.53 (PC0); no longer U2.56 (PC3)
- net SLEEP_STP2: now also U2.55 (PC2); no longer U2.57 (PC4)
- net SLEEP_STP3: now also U2.57 (PC4); no longer U2.58 (PC5)
- net VM: now also J1.2
Other:
- moved on the sheet: J1

Commit message: Correct JST header footprint and minor silkscreen changes
Parts:
- STP1_OUT1, STP2_OUT1, STP3_OUT1: footprint Connector_PinHeader_2.54mm:PinHeader_1x04_P2.54mm_Vertical -> Connector_JST:JST_XH_B4B-XH-A_1x04_P2.50mm_Vertical
Connections:
- net AOUT1_STP1: now also STP1_OUT1.4 (Pin_4); no longer STP1_OUT1.1 (Pin_1)
- net AOUT1_STP2: now also STP2_OUT1.4 (Pin_4); no longer STP2_OUT1.1 (Pin_1)
- net AOUT1_STP3: now also STP3_OUT1.4 (Pin_4); no longer STP3_OUT1.1 (Pin_1)
- net AOUT2_STP1: now also STP1_OUT1.3 (Pin_3); no longer STP1_OUT1.2 (Pin_2)
- net AOUT2_STP2: now also STP2_OUT1.3 (Pin_3); no longer STP2_OUT1.2 (Pin_2)
- net AOUT2_STP3: now also STP3_OUT1.3 (Pin_3); no longer STP3_OUT1.2 (Pin_2)
- net BOUT1_STP1: now also STP1_OUT1.1 (Pin_1); no longer STP1_OUT1.4 (Pin_4)
- net BOUT1_STP2: now also STP2_OUT1.1 (Pin_1); no longer STP2_OUT1.4 (Pin_4)
- net BOUT1_STP3: now also STP3_OUT1.1 (Pin_1); no longer STP3_OUT1.4 (Pin_4)
- net BOUT2_STP1: now also STP1_OUT1.2 (Pin_2); no longer STP1_OUT1.3 (Pin_3)
- net BOUT2_STP2: now also STP2_OUT1.2 (Pin_2); no longer STP2_OUT1.3 (Pin_3)
- net BOUT2_STP3: now also STP3_OUT1.2 (Pin_2); no longer STP3_OUT1.3 (Pin_3)
Other:
- moved on the sheet: STP1_OUT1
Changed lines of the file:
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@@
 	(wire
 		(pts
+			(xy 147.32 137.16) (xy 153.67 137.16)
+		)
+		(stroke
+			(width 0)
+			(type default)
+		)
+	)
+	(wire
+		(pts
 			(xy 213.36 236.22) (xy 213.36 234.95)
 		)
@@
 	(wire
 		(pts
+			(xy 148.59 158.75) (xy 153.67 158.75)
+		)
+		(stroke
+			(width 0)
+			(type default)
+		)
+	)
+	(wire
+		(pts
 			(xy 186.69 198.12) (xy 194.31 198.12)
 		)
@@
 	(wire
 		(pts
-			(xy 148.59 142.24) (xy 153.67 142.24)
-		)
-		(stroke
-			(width 0)
-			(type default)
-		)
-	)
-	(wire
-		(pts
 			(xy 46.99 257.81) (xy 46.99 264.16)
 		)
@@
 	(wire
 		(pts
+			(xy 147.32 142.24) (xy 153.67 142.24)
+		)
+		(stroke
+			(width 0)
+			(type default)
+		)
+	)
+	(wire
+		(pts
 			(xy 48.26 123.19) (xy 50.8 123.19)
 		)
@@
 	(wire
 		(pts
+			(xy 148.59 171.45) (xy 153.67 171.45)
+		)
+		(stroke
+			(width 0)
+			(type default)
+		)
+	)
+	(wire
+		(pts
 			(xy 60.96 257.81) (xy 60.96 264.16)
 		)
@@
 	(wire
 		(pts
+			(xy 148.59 156.21) (xy 153.67 156.21)
+		)
+		(stroke
+			(width 0)
+			(type default)
+		)
+	)
+	(wire
+		(pts
 			(xy 200.66 233.68) (xy 203.2 233.68)
 		)
@@
 	(wire
 		(pts
+			(xy 147.32 134.62) (xy 153.67 134.62)
+		)
+		(stroke
+			(width 0)
+			(type default)
+		)
+	)
+	(wire
+		(pts
 			(xy 229.87 139.7) (xy 241.3 139.7)
 		)
@@
 	(wire
 		(pts
-			(xy 148.59 158.75) (xy 153.67 158.75)
-		)
-		(stroke
-			(width 0)
-			(type default)
-		)
-	)
-	(wire
-		(pts
 			(xy 48.26 189.23) (xy 48.26 186.69)
 		)
@@
 	(wire
 		(pts
-			(xy 148.59 139.7) (xy 153.67 139.7)
-		)
-		(stroke
-			(width 0)
-			(type default)
-		)
-	)
-	(wire
-		(pts
 			(xy 96.52 125.73) (xy 99.06 125.73)
 		)
@@
 	(wire
 		(pts
-			(xy 148.59 137.16) (xy 153.67 137.16)
-		)
-		(stroke
-			(width 0)
-			(type default)
-		)
-	)
-	(wire
-		(pts
 			(xy 281.94 187.96) (xy 295.91 187.96)
 		)
@@
 	(wire
 		(pts
-			(xy 148.59 134.62) (xy 153.67 134.62)
+			(xy 147.32 139.7) (xy 153.67 139.7)
 		)
 		(stroke
@@
 		)
 	)
-	(wire
-		(pts
-			(xy 148.59 176.53) (xy 153.67 176.53)
-		)
-		(stroke
-			(width 0)
-			(type default)
-		)
-	)
 	(polyline
 		(pts
@@
 	(wire
 		(pts
+			(xy 148.59 168.91) (xy 153.67 168.91)
+		)
+		(stroke
+			(width 0)
+			(type default)
+		)
+	)
+	(wire
+		(pts
 			(xy 22.86 236.22) (xy 35.56 236.22)
 		)
@@
 	(wire
 		(pts
+			(xy 148.59 173.99) (xy 153.67 173.99)
+		)
+		(stroke
+			(width 0)
+			(type default)
+		)
+	)
+	(wire
+		(pts
 			(xy 200.66 184.15) (xy 207.01 184.15)
 		)
@@
 	(wire
 		(pts
+			(xy 148.59 176.53) (xy 153.67 176.53)
+		)
+		(stroke
+			(width 0)
+			(type default)
+		)
+	)
+	(wire
+		(pts
 			(xy 245.11 77.47) (xy 245.11 78.74)
 		)
@@
 	(wire
 		(pts
-			(xy 148.59 153.67) (xy 153.67 153.67)
-		)
-		(stroke
-			(width 0)
-			(type default)
-		)
-	)
-	(wire
-		(pts
 			(xy 190.5 238.76) (xy 186.69 238.76)
 		)
@@
 	(wire
 		(pts
+			(xy 148.59 153.67) (xy 153.67 153.67)
+		)
+		(stroke
+			(width 0)
+			(type default)
+		)
+	)
+	(wire
+		(pts
 			(xy 34.29 130.81) (xy 48.26 130.81)
 		)
@@
 	(wire
 		(pts
-			(xy 148.59 171.45) (xy 153.67 171.45)
-		)
-		(stroke
-			(width 0)
-			(type default)
-		)
-	)
-	(wire
-		(pts
 			(xy 281.94 160.02) (xy 295.91 160.02)
 		)
@@
 	(wire
 		(pts
-			(xy 148.59 156.21) (xy 153.67 156.21)
-		)
-		(stroke
-			(width 0)
-			(type default)
-		)
-	)
-	(wire
-		(pts
 			(xy 48.26 236.22) (xy 58.42 236.22)
 		)
@@
 	(wire
 		(pts
-			(xy 148.59 151.13) (xy 153.67 151.13)
-		)
-		(stroke
-			(width 0)
-			(type default)
-		)
-	)
-	(wire
-		(pts
 			(xy 281.94 172.72) (xy 295.91 172.72)
 		)
@@
 	(wire
 		(pts
-			(xy 148.59 173.99) (xy 153.67 173.99)
-		)
-		(stroke
-			(width 0)
-			(type default)
-		)
-	)
-	(wire
-		(pts
 			(xy 19.05 274.32) (xy 33.02 274.32)
 		)
@@
 	(wire
 		(pts
-			(xy 148.59 168.91) (xy 153.67 168.91)
-		)
-		(stroke
-			(width 0)
-			(type default)
-		)
-	)
-	(wire
-		(pts
 			(xy 38.1 100.33) (xy 50.8 100.33)
 		)
@@
 	(wire
 		(pts
+			(xy 148.59 151.13) (xy 153.67 151.13)
+		)
+		(stroke
+			(width 0)
+			(type default)
+		)
+	)
+	(wire
+		(pts
 			(xy 138.43 83.82) (xy 137.16 83.82)
 		)
@@
 	(symbol
 		(lib_id "Connector:Conn_01x04_Pin")
-		(at 143.51 153.67 0)
+		(at 143.51 156.21 0)
+		(mirror x)
 		(unit 1)
 		(exclude_from_sim no)
@@
 		(dnp no)
 		(property "Reference" "STP3_OUT1"
-			(at 142.24 153.6699 0)
+			(at 142.24 156.2101 0)
 			(effects
 				(font
@@
 		)
 		(property "Value" "STP3_OUT"
-			(at 142.24 156.2099 0)
+			(at 142.24 153.6701 0)
 			(effects
 				(font
@@
 			)
 		)
-		(property "Footprint" "Connector_PinHeader_2.54mm:PinHeader_1x04_P2.54mm_Vertical"
-			(at 143.51 153.67 0)
+		(property "Footprint" "Connector_JST:JST_XH_B4B-XH-A_1x04_P2.50mm_Vertical"
+			(at 143.51 156.21 0)
 			(effects
 				(font
@@
 		)
 		(property "Datasheet" "~"
-			(at 143.51 153.67 0)
+			(at 143.51 156.21 0)
 			(effects
 				(font
@@
 		)
 		(property "Description" "Generic connector, single row, 01x04, script generated"
-			(at 143.51 153.67 0)
+			(at 143.51 156.21 0)
 			(effects
 				(font
@@
 	(symbol
 		(lib_id "Connector:Conn_01x04_Pin")
-		(at 143.51 171.45 0)
+		(at 143.51 173.99 0)
+		(mirror x)
 		(unit 1)
 		(exclude_from_sim no)
@@
 		(dnp no)
 		(property "Reference" "STP2_OUT1"
-			(at 142.24 171.4499 0)
+			(at 142.24 173.9901 0)
 			(effects
 				(font
@@
 		)
 		(property "Value" "STP2_OUT"
-			(at 142.24 173.9899 0)
+			(at 142.24 171.4501 0)
 			(effects
 				(font
@@
 			)
 		)
-		(property "Footprint" "Connector_PinHeader_2.54mm:PinHeader_1x04_P2.54mm_Vertical"
-			(at 143.51 171.45 0)
+		(property "Footprint" "Connector_JST:JST_XH_B4B-XH-A_1x04_P2.50mm_Vertical"
+			(at 143.51 173.99 0)
 			(effects
 				(font
@@
 		)
 		(property "Datasheet" "~"
-			(at 143.51 171.45 0)
+			(at 143.51 173.99 0)
 			(effects
 				(font
@@
 		)
 		(property "Description" "Generic connector, single row, 01x04, script generated"
-			(at 143.51 171.45 0)
+			(at 143.51 173.99 0)
 			(effects
 				(font
@@
 	(symbol
 		(lib_id "Connector:Conn_01x04_Pin")
-		(at 143.51 137.16 0)
+		(at 142.24 139.7 0)
+		(mirror x)
 		(unit 1)
 		(exclude_from_sim no)
@@
 		(dnp no)
 		(property "Reference" "STP1_OUT1"
-			(at 142.24 137.1599 0)
+			(at 140.97 139.7001 0)
 			(effects
 				(font
@@
 		)
 		(property "Value" "STP1_OUT"
-			(at 142.24 139.6999 0)
+			(at 140.97 137.1601 0)
 			(effects
 				(font
@@
 			)
 		)
-		(property "Footprint" "Connector_PinHeader_2.54mm:PinHeader_1x04_P2.54mm_Vertical"
-			(at 143.51 137.16 0)
+		(property "Footprint" "Connector_JST:JST_XH_B4B-XH-A_1x04_P2.50mm_Vertical"
+			(at 142.24 139.7 0)
 			(effects
 				(font
@@
 		)
 		(property "Datasheet" "~"
-			(at 143.51 137.16 0)
+			(at 142.24 139.7 0)
 			(effects
 				(font
@@
 		)
 		(property "Description" "Generic connector, single row, 01x04, script generated"
-			(at 143.51 137.16 0)
+			(at 142.24 139.7 0)
 			(effects
 				(font
